File: 0002_Accelerometer_Module_ADXL345.kicad_sch (KiCad schematic)
At the start: 6 parts, among them U1 ADXL345BCCZ

Commit message: Add files via upload
Parts:
- removed C1: 10uF, Capacitor_Tantalum_SMD:CP_EIA-3216-10_Kemet-I, symbol Device:C_Polarized_Small_US
- added D1: LED, LED_SMD:LED_0805_2012Metric, symbol Device:LED
- added R3, R4: 4.7k, Resistor_SMD:R_0805_2012Metric, symbol Device:R
- added R5: 470r, Resistor_SMD:R_0805_2012Metric, symbol Device:R
- added U3: ~, Moduler_:pin_header, symbol moduler_pin:air
- C1: renamed from C3; footprint Capacitor_SMD:C_0603_1608Metric -> Capacitor_SMD:C_0805_2012Metric
- C2: footprint Capacitor_SMD:C_0603_1608Metric -> Capacitor_SMD:C_0805_2012Metric
- R1, R2: footprint Resistor_SMD:R_0603_1608Metric -> Resistor_SMD:R_0805_2012Metric
Connections:
- net +3V3: now also R3.1, R5.1, U3.8
- net CS: now also R3.2, U3.3
- net GND: now also D1.1 (K), R4.2, U3.9
- net INT1: now also U3.12
- net INT2: now also U3.13
- net SCL: now also U3.5
- net SD0: now also R4.1, U3.2
- net SDA: now also U3.6
- new net: D1.2 (A), R5.2
- no-connect marks 2 -> 12
Other:
- note added: "AIR PIN"
- note added: "I2C PULLUPS"
- note added: "SENSOR"
- moved on the sheet: C1, C2, R1, R2, U1
